File: PCB/TWPad.kicad_pcb (KiCad board)
At the start: 2 copper layers, 97.6 x 66.7 mm, 31 parts, among them SW1 RotaryEncoder_Switch, SW3 RotaryEncoder_Switch, U1 MCU_Seeed_XIAO_RP2040, U2 SN74LV1T34DBV

Commit message: Adding necesary files/updating them for cad and pcb
Parts:
- removed U2: SN74LV1T34DBV, Package_TO_SOT_SMD:SOT-23-5
Other:
- board text added: "RP Here"
- board text added: "TWPad by JFKB"
